File: Esp32_Emircan/Emircan_ESP32.kicad_sch (KiCad schematic)
At the start: 34 parts, among them J1 Conn_01x04_Female, J2 Conn_01x02_Female, J3 Conn_01x04_Female, SW1 SW_DPST_x2, U1 PCM5100, U2 ESP32-WROOM-32U, Y1 Crystal

Commit message: Update Emircan_ESP32.kicad_sch
Parts:
- C1, C5, C8: footprint (none) -> Capacitor_SMD:CP_Elec_3x5.3
- C11, C12, C13, C14, C15, C16, C17, C18, C2, C3, C30, C4, C6, C7, C9: footprint (none) -> Capacitor_SMD:C_0805_2012Metric
- J1, J3: footprint (none) -> Connector_PinSocket_1.00mm:PinSocket_1x04_P1.00mm_Vertical
- J2: footprint (none) -> Connector_PinSocket_1.00mm:PinSocket_1x02_P1.00mm_Vertical
- JP6: footprint (none) -> TestPoint:TestPoint_2Pads_Pitch2.54mm_Drill0.8mm
- R1, R2, R3, R4, R5, R6, R7, R8: footprint (none) -> Resistor_SMD:R_0805_2012Metric
- Y1: footprint (none) -> Crystal:Crystal_AT310_D3.0mm_L10.0mm_Vertical
